File: hw/picocart64_v2/overview.kicad_sch (KiCad schematic)
At the start: 0 parts

Commit message: hw: v2 Finalize schematic
Other:
- note added: "0 ESP32_GP9/ROMBL [reuse QSPI pins]"
- note added: "0 UART [reuse QSPI pins]"
- note added: "Debug UART"
- note added: "MCU2 Clock output"
- note added: "MCU2 Pin Count = 30 4+1+3+1+1+2+1 + 1+2+1+6+6+1"
- note removed: "0 [reuse QSPI pins for UART]"
- note removed: "1 ESP32_GP9/ROMBL"
- note removed: "MCU2 Pin Count = 28 4+1+3+1+1+2+1+1+6+1+6+1"
