File: hw/picocart64_v2/picocart64_v2.kicad_sch (KiCad schematic)
At the start: 16 parts, among them J1 USB_C_Receptacle_USB2.0, J2 Conn_01x05, J3 Conn_02x06_Odd_Even, J4 Micro_SD_Card_Det, Q1 BSS84, SW1 BootButton, U3 RP2040_Stamp, U4 N64-Cartridge

Commit message: hw: v2 WIP
Parts:
- removed J2: Conn_01x05, Connector_PinHeader_2.54mm:PinHeader_1x05_P2.54mm_Vertical, symbol Connector_Generic:Conn_01x05
- removed J3: Conn_02x06_Odd_Even, Connector_PinSocket_2.54mm:PinSocket_2x06_P2.54mm_Horizontal, symbol Connector_Generic:Conn_02x06_Odd_Even
- removed JP1, JP2, JP3, JP4: SolderJumper_2_Open, Jumper:SolderJumper-2_P1.3mm_Open_TrianglePad1.0x1.5mm, symbol Jumper:SolderJumper_2_Open
- removed Q1: BSS84, Package_TO_SOT_SMD:SOT-23, symbol Transistor_FET:BSS84
- removed U3: RP2040_Stamp, RP2040_Stamp:RP2040_Stamp_FlexyPin, symbol RP2040_Stamp:RP2040_Stamp
- removed U4: N64-Cartridge, picocart64:N64-Connector, symbol n64-cartridge:N64-Cartridge
- added C? (x17): 100n, symbol Device:C_Small
- added C? (x4): 1u, symbol Device:C_Small
- added C? (x4): 12p, symbol Device:C_Small
- added C?: 22u, symbol Device:C_Small
- added C?: 10u7, symbol Device:C_Small
- added J?: Conn_01x10, symbol Connector_Generic:Conn_01x10
- added J?: USB_C_Receptacle_USB2.0, Connector_USB_Extra:USB_C_Receptacle_GT-USB-7010, symbol Connector:USB_C_Receptacle_USB2.0
- added Q?: FDN340P, Package_TO_SOT_SMD:SOT-23, symbol Transistor_FET:FDN340P
- added R? (x4): 10K, symbol Device:R_Small
- added R? (x4): 22R, symbol Device:R_Small
- added R? (x2): 22R, symbol Device:R
- added R?: 1K, symbol Device:R_Small
- added R?: 0R, symbol Device:R_Small
- added R?: 1M, Resistor_SMD:R_0603_1608Metric, symbol Device:R_Small
- added RN? (x6): 22R_x4, Resistor_SMD:R_Array_Convex_4x0603, symbol Device:R_Pack04
- added TP? (x2): TP_MCU2_CS, symbol Connector:TestPoint
- added TP?: MCU2_DIO, symbol Connector:TestPoint
- added U?: N64-Cartridge, picocart64:N64-Connector, symbol n64-cartridge:N64-Cartridge
- added U? (x2): RP2040, Package_DFN_QFN_Extra:QFN-56_EP_7x7_Pitch0.4mm, symbol MCU_RaspberryPi:RP2040
- added U?: W25Q128JVS, Package_SO:SOIC-8_5.23x5.23mm_P1.27mm, symbol Memory_Flash:W25Q128JVS
- added U?: AZ1117-3.3, symbol Regulator_Linear:AZ1117-3.3
- added U?: USBLC6-2SC6, Package_TO_SOT_SMD:SOT-23-6, symbol Power_Protection:USBLC6-2SC6
- added Y? (x2): 12MHz 10ppm, symbol Device:Crystal_GND24_Small
- renumbered FB1 to FB?, J4 to J?, J1 to J?, R1 to R?, R3 to R?, R2 to R?, SW1 to SW?
Connections:
- net +3V3: now also C?.1, C?.1, C?.1, C?.1, C?.1, C?.1, C?.1, C?.1, C?.1, C?.1, C?.1, C?.1, C?.1, C?.1, C?.1, C?.1, J?.10 (Pin_10), J?.4 (Pin_4), Q?.2 (S), R?.1, R?.1, R?.1, U?.1 (IOVDD), U?.1 (IOVDD), U?.10 (IOVDD), U?.10 (IOVDD), U?.22 (IOVDD), U?.22 (IOVDD), U?.33 (IOVDD), U?.33 (IOVDD), U?.42 (IOVDD), U?.42 (IOVDD), U?.43 (ADC_AVDD), U?.43 (ADC_AVDD), U?.44 (VREG_VIN), U?.44 (VREG_VIN), U?.48 (USB_VDD), U?.48 (USB_VDD), U?.49 (IOVDD), U?.49 (IOVDD), U?.8 (VCC)
- net AD0: now also RN?.8 (R1.2), U?.2 (GPIO0)
- net AD1: now also RN?.7 (R2.2), U?.3 (GPIO1)
- net AD10: now also RN?.4 (R4.1), U?.13 (GPIO10)
- net AD11: now also RN?.3 (R3.1), U?.14 (GPIO11)
- net AD12: now also RN?.4 (R4.1), U?.15 (GPIO12)
- net AD13: now also RN?.3 (R3.1), U?.16 (GPIO13)
- net AD14: now also RN?.2 (R2.1), U?.17 (GPIO14)
- net AD15: now also RN?.1 (R1.1), U?.18 (GPIO15)
- net AD2: now also RN?.6 (R3.2), U?.4 (GPIO2)
- net AD3: now also RN?.5 (R4.2), U?.5 (GPIO3)
- net AD4: now also RN?.6 (R3.2), U?.6 (GPIO4)
- net AD5: now also RN?.5 (R4.2), U?.7 (GPIO5)
- net AD6: now also RN?.8 (R1.2), U?.8 (GPIO6)
- net AD7: now also RN?.7 (R2.2), U?.9 (GPIO7)
- net AD8: now also RN?.2 (R2.1), U?.11 (GPIO8)
- net AD9: now also RN?.1 (R1.1), U?.12 (GPIO9)
- net ALEH: now also RN?.7 (R2.2), U?.28 (GPIO17)
- net ALEL: now also RN?.8 (R1.2), U?.27 (GPIO16)
- net GND: now also C?.1, C?.1, C?.1, C?.1, C?.2, C?.2, C?.2, C?.2, C?.2, C?.2, C?.2, C?.2, C?.2, C?.2, C?.2, C?.2, C?.2, C?.2, C?.2, C?.2, C?.2, C?.2, C?.2, C?.2, C?.2, C?.2, C?.2, J?.9 (Pin_9), J?.A1 (GND), J?.A12 (GND), J?.B1 (GND), J?.B12 (GND), R?.1, R?.1, R?.2, U?.1 (GND), U?.1 (GND), U?.19 (TESTEN), U?.19 (TESTEN), U?.2 (GND), U?.2 (GND), U?.22 (GND), U?.23 (GND), U?.25 (GND), U?.26 (GND), U?.27 (GND), U?.31 (GND), U?.4 (GND), U?.47 (GND), U?.48 (GND), U?.50 (GND), U?.57 (GND), U?.57 (GND), U?.6 (GND), Y?.2, Y?.2, Y?.4, Y?.4; no longer SW?.1
- net N64_VCC: now also Q?.3 (D), U?.17 (VCC), U?.34 (VCC), U?.42 (VCC), U?.9 (VCC)
- net VBUS: now also C?.1, U?.3 (VI), U?.5 (VBUS)
- net ~{READ}: now also RN?.2 (R2.1), U?.30 (GPIO19)
- net ~{WRITE}: now also RN?.1 (R1.1), U?.29 (GPIO18)
- net at SW?.2: now also R?.1
- net PMOD_1_SS renamed SD_CMD
- net SD_CMD: now also U?.5 (GPIO3)
- net PMOD_2_SIO0 renamed SD_DAT0
- net SD_DAT0: now also U?.6 (GPIO4)
- net PMOD_3_SIO1 renamed SD_DAT1
- net SD_DAT1: now also U?.7 (GPIO5)
- net PMOD_4_SCLK renamed SD_CLK
- net SD_CLK: now also U?.4 (GPIO2)
- net PMOD_5_SIO2 renamed SD_DAT2
- net SD_DAT2: now also U?.8 (GPIO6)
- net PMOD_6_SIO3 renamed SD_DAT3
- net SD_DAT3: now also U?.9 (GPIO7)
- net PMOD_7_CS0 renamed SD_DET
- net USB_D+ renamed MCU2_USB_D+
- net MCU2_USB_D+: now also R?.1, U?.3 (I/O2), U?.4 (I/O2)
- net USB_D- renamed MCU2_USB_D-
- net MCU2_USB_D-: now also R?.1, U?.1 (I/O1), U?.6 (I/O1)
- net VBUS_unf renamed VBUS'
- new net: C?.1, C?.1, C?.1, U?.23 (DVDD), U?.45 (VREG_VOUT), U?.50 (DVDD) (x2)
- new net: R?.2, U?.46 (USB_D-) (x2)
- new net: C?.2, U?.21 (XOUT), Y?.1 (x2)
- new net: C?.2, U?.20 (XIN), Y?.3 (x2)
- new net: R?.2, U?.47 (USB_D+) (x2)
- new net: R?.2, U?.26 (RUN)
- new net: J?.A4 (VBUS), J?.A9 (VBUS), J?.B4 (VBUS), J?.B9 (VBUS)
- new net: J?.S1 (SHIELD), R?.2
- new net: R?.1, U?.39 (GPIO27)
- new net 3V3_USB: Q?.1 (G), U?.2 (VO)
- new net AD0': RN?.1 (R1.1), U?.28 (AD0)
- new net AD1': RN?.2 (R2.1), U?.29 (AD1)
- new net AD10': RN?.5 (R4.2), U?.12 (AD10)
- new net AD11': RN?.6 (R3.2), U?.11 (AD11)
- new net AD12': RN?.5 (R4.2), U?.7 (AD12)
- new net AD13': RN?.6 (R3.2), U?.5 (AD13)
- new net AD14': RN?.7 (R2.2), U?.4 (AD14)
- new net AD15': RN?.8 (R1.2), U?.3 (AD15)
- new net AD2': RN?.3 (R3.1), U?.30 (AD2)
- new net AD3': RN?.4 (R4.1), U?.32 (AD3)
- new net AD4': RN?.3 (R3.1), U?.36 (AD4)
- new net AD5': RN?.4 (R4.1), U?.37 (AD5)
- new net AD6': RN?.1 (R1.1), U?.40 (AD6)
- new net AD7': RN?.2 (R2.1), U?.41 (AD7)
- new net AD8': RN?.7 (R2.2), U?.16 (AD8)
- new net AD9': RN?.8 (R1.2), U?.15 (AD9)
- new net ALEH': RN?.2 (R2.1), U?.35 (ALEH)
- new net ALEL': RN?.1 (R1.1), U?.33 (ALEL)
- new net CIC_DCLK: RN?.6 (R3.2)
- new net CIC_DCLK': RN?.3 (R3.1), U?.43 (CIC_DCLK)
- new net CIC_DIO: RN?.3 (R3.1)
- new net CIC_DIO': RN?.6 (R3.2), U?.18 (CIC_DIO)
- new net DEMUX_A0: U?.35 (GPIO23)
- new net DEMUX_A1: U?.36 (GPIO24)
- new net DEMUX_A2: U?.37 (GPIO25)
- new net DEMUX_IE: U?.38 (GPIO26)
- new net MCU1_RUN: J?.8 (Pin_8), R?.2, U?.26 (RUN)
- new net MCU1_SWCLK: J?.7 (Pin_7), U?.24 (SWCLK)
- new net MCU1_SWDIO: J?.6 (Pin_6), U?.25 (SWDIO)
- new net MCU1_USB_D+: J?.A6 (D+), J?.B6 (D+), R?.1
- new net MCU1_USB_D-: J?.A7 (D-), J?.B7 (D-), R?.1
- new net MCU2_CS: J?.5 (Pin_5), R?.2, TP?.1, U?.40 (GPIO28), U?.41 (GPIO29)
- new net MCU2_DIO: R?.2, TP?.1, U?.40 (GPIO28), U?.41 (GPIO29)
- new net MCU2_SCK: TP?.1, U?.38 (GPIO26), U?.39 (GPIO27)
- new net MCU2_SWCLK: J?.3 (Pin_3), U?.24 (SWCLK)
- new net MCU2_SWDIO: J?.2 (Pin_2), U?.25 (SWDIO)
- new net MCU2_UART_TX: J?.1 (Pin_1)
- new net SI_CLK: U?.19 (SI_CLK)
- new net SI_DAT: R?.1, U?.32 (GPIO21)
- new net SI_DAT': R?.2, U?.21 (SI_DAT)
- new net SSI_SCLK: U?.52 (QSPI_SCLK), U?.52 (QSPI_SCLK), U?.6 (CLK)
- new net SSI_SD0: U?.5 (DI(IO0)), U?.53 (QSPI_SD0), U?.53 (QSPI_SD0)
- new net SSI_SD1: U?.2 (DO(IO1)), U?.55 (QSPI_SD1), U?.55 (QSPI_SD1)
- new net SSI_SD2: U?.3 (IO2), U?.54 (QSPI_SD2), U?.54 (QSPI_SD2)
- new net SSI_SD3: U?.51 (QSPI_SD3), U?.51 (QSPI_SD3), U?.7 (IO3)
- new net ~{COLD_RESET'}: RN?.5 (R4.2), U?.20 (~{COLD_RESET})
- new net ~{COLD_RESET}: RN?.4 (R4.1), U?.31 (GPIO20)
- new net ~{INT1'}: RN?.4 (R4.1), U?.44 (~{INT1})
- new net ~{INT1}: RN?.5 (R4.2), U?.34 (GPIO22)
- new net ~{NMI'}: R?.1, U?.45 (~{NMI})
- new net ~{NMI}: R?.2
- new net ~{READ'}: RN?.7 (R2.2), U?.10 (~{READ})
- new net ~{SSI_CS}: R?.2, SW?.1, U?.1 (~{CS}), U?.56 (~{QSPI_CS}), U?.56 (~{QSPI_CS})
- new net ~{WRITE'}: RN?.8 (R1.2), U?.8 (~{WRITE})
- no-connect marks 11 -> 15
Other:
- added sheet PSRAM Array (psram.kicad_sch)
- note added: "Compatible with many LDOs"
- note added: "DNP - For extra debug/evaluation only CC resistors omitted for simplicity"
- note added: "Either use SPI0 with custom CS pin, or do QSPI with PIO"
- note added: "FDN340P is rated for 2A Prevent N64_VCC to feed into LDO Prevent 3V3_USB to feed into N64_VCC If both are connected, pick 3V3_USB"
- note added: "MCU1 <-> MCU2 communication 1. If possible, try SSI + MCU2_CS. Need to implement slave mode on MCU2 2. Backup solution, use SPI (PIO on MCU1, SPI slave on MCU2) 3. Backup solution, use SPI (PIO on MCU1, PIO on MCU2) 4. Backup solution, use UART MCU2_CS might function as MCU1_INT."
- note added: "MCU1 Handles the N64_BUS"
- note added: "MCU2 Handles ESP32, SDCard"
- note added: "MCU2 USB connector"
- note added: "NOTE: MCU2 will drive pin high"
- note added: "NOTE: MCU2_DIO and MCU2_CS are connected UART as well (backup solution)"
- note added: "NOTE: May switch to smaller flash later. Let's go for 16MB, makes it easier to develop."
- note added: "Optional ESD protection"
- note added: "Strong pull"
- note added: "TODO: Add ESP32-C3-WROOM-02-H4"
- note added: "TODO: Carefully pick GPIO to identify MCU1/MCU2"
- note added: "TODO: Do we need ESD protection?"
- note added: "TODO: Figure out if we want to use 0402 or 0603 resistor arrays"
- note added: "TODO: Hook up ESP32 signals"
- note added: "[MCU1_UART_TX]"
- note added: "[PIO0_IO2]"
- note added: "[PIO0_IO3]"
- note added: "[Pulled Down]"
- note added: "[Pulled Up]"
- note added: "[SPI0_RX/MISO/PIO0_IO1]"
- note added: "[SPI0_SCK]"
- note added: "[SPI0_TX/MOSI/PIO0_IO0]"
- note added: "[SPI1_CSn]"
- note added: "[SPI1_RX]"
- note added: "[SPI1_SCK]"
- note added: "[SPI1_TX]"
- note added: "[UART0_RX -> MCU2_TX]"
- note added: "[UART0_RX]"
- note added: "[UART0_TX -> MCU2_RX]"
- note added: "[UART0_TX]"
- note added: "[gpio_CSn/PIO0_IO4]"
- note removed: "Absolute minimum"
- note removed: "Not enough I/Os to handle these"
- note removed: "Power from USB if possible, N64_VCC otherwise. N64_VCC is disconnected if USB powered."
- moved on the sheet: FB?, J?, R?, SW?

Commit message: Break out sheets
Parts:
- removed C? (x17): 100n, symbol Device:C_Small
- removed C? (x4): 1u, symbol Device:C_Small
- removed C? (x4): 12p, symbol Device:C_Small
- removed C?: 22u, symbol Device:C_Small
- removed C?: 10u7, symbol Device:C_Small
- removed FB?: Ferrite, Inductor_SMD:L_0603_1608Metric, symbol Device:FerriteBead_Small
- removed J?: Micro_SD_Card_Det, Connector_Card:microSD_HC_Molex_104031-0811, symbol Connector:Micro_SD_Card_Det
- removed J?: Conn_01x10, symbol Connector_Generic:Conn_01x10
- removed J? (x2): USB_C_Receptacle_USB2.0, Connector_USB_Extra:USB_C_Receptacle_GT-USB-7010, symbol Connector:USB_C_Receptacle_USB2.0
- removed Q?: FDN340P, Package_TO_SOT_SMD:SOT-23, symbol Transistor_FET:FDN340P
- removed R? (x4): 10K, symbol Device:R_Small
- removed R? (x4): 22R, symbol Device:R_Small
- removed R? (x2): 1M, Resistor_SMD:R_0603_1608Metric, symbol Device:R_Small
- removed R? (x2): 22R, symbol Device:R
- removed R?: 1K, symbol Device:R_Small
- removed R?: 0R, symbol Device:R_Small
- removed R? (x2): 5k1, Resistor_SMD:R_0603_1608Metric, symbol Device:R_Small
- removed RN? (x6): 22R_x4, Resistor_SMD:R_Array_Convex_4x0603, symbol Device:R_Pack04
- removed SW?: BootButton, Button_Switch_SMD:SW_SPST_FSMSM, symbol Switch:SW_Push
- removed TP? (x2): TP_MCU2_CS, symbol Connector:TestPoint
- removed TP?: MCU2_DIO, symbol Connector:TestPoint
- removed U?: N64-Cartridge, picocart64:N64-Connector, symbol n64-cartridge:N64-Cartridge
- removed U? (x2): RP2040, Package_DFN_QFN_Extra:QFN-56_EP_7x7_Pitch0.4mm, symbol MCU_RaspberryPi:RP2040
- removed U?: W25Q128JVS, Package_SO:SOIC-8_5.23x5.23mm_P1.27mm, symbol Memory_Flash:W25Q128JVS
- removed U?: AZ1117-3.3, symbol Regulator_Linear:AZ1117-3.3
- removed U?: USBLC6-2SC6, Package_TO_SOT_SMD:SOT-23-6, symbol Power_Protection:USBLC6-2SC6
- removed Y? (x2): 12MHz 10ppm, symbol Device:Crystal_GND24_Small
Connections:
- no-connect marks 15 -> 0
Other:
- added sheet Mainboard (board.kicad_sch)
- note removed: "Compatible with many LDOs"
- note removed: "DNP - For extra debug/evaluation only CC resistors omitted for simplicity"
- note removed: "Either use SPI0 with custom CS pin, or do QSPI with PIO"
- note removed: "FDN340P is rated for 2A Prevent N64_VCC to feed into LDO Prevent 3V3_USB to feed into N64_VCC If both are connected, pick 3V3_USB"
- note removed: "MCU1 <-> MCU2 communication 1. If possible, try SSI + MCU2_CS. Need to implement slave mode on MCU2 2. Backup solution, use SPI (PIO on MCU1, SPI slave on MCU2) 3. Backup solution, use SPI (PIO on MCU1, PIO on MCU2) 4. Backup solution, use UART MCU2_CS might function as MCU1_INT."
- note removed: "MCU1 Handles the N64_BUS"
- note removed: "MCU2 Handles ESP32, SDCard"
- note removed: "MCU2 USB connector"
- note removed: "NOTE: MCU2 will drive pin high"
- note removed: "NOTE: MCU2_DIO and MCU2_CS are connected UART as well (backup solution)"
- note removed: "NOTE: May switch to smaller flash later. Let's go for 16MB, makes it easier to develop."
- note removed: "Optional ESD protection"
- note removed: "Strong pull"
- note removed: "TODO: Add ESP32-C3-WROOM-02-H4"
- note removed: "TODO: Carefully pick GPIO to identify MCU1/MCU2"
- note removed: "TODO: Do we need ESD protection?"
- note removed: "TODO: Figure out if we want to use 0402 or 0603 resistor arrays"
- note removed: "TODO: Hook up ESP32 signals"
- note removed: "[MCU1_UART_TX]"
- note removed: "[PIO0_IO2]"
- note removed: "[PIO0_IO3]"
- note removed: "[Pulled Down]"
- note removed: "[Pulled Up]"
- note removed: "[SPI0_RX/MISO/PIO0_IO1]"
- note removed: "[SPI0_SCK]"
- note removed: "[SPI0_TX/MOSI/PIO0_IO0]"
- note removed: "[SPI1_CSn]"
- note removed: "[SPI1_RX]"
- note removed: "[SPI1_SCK]"
- note removed: "[SPI1_TX]"
- note removed: "[UART0_RX -> MCU2_TX]"
- note removed: "[UART0_RX]"
- note removed: "[UART0_TX -> MCU2_RX]"
- note removed: "[UART0_TX]"
- note removed: "[gpio_CSn/PIO0_IO4]"

Commit message: Add overview
Other:
- added sheet overview (overview.kicad_sch)
Changed lines of the file:
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@@
+    )
+  )
+  (sheet (at 111.76 38.735) (size 61.595 21.59) (fields_autoplaced)
+    (stroke (width 0.1524) (type solid) (color 0 0 0 0))
+    (fill (color 0 0 0 0.0000))
+    (property "Sheet name" "overview" (id 0) (at 111.76 38.0234 0)
+      (effects (font (size 1.27 1.27)) (justify left bottom))
+    )
+    (property "Sheet file" "overview.kicad_sch" (id 1) (at 111.76 60.9096 0)
+      (effects (font (size 1.27 1.27)) (justify left top))
     )
   )
@@
     (path "/18bc2029-d732-4df0-8cd4-b3abe43b5862" (page "2"))
     (path "/a45f4a80-c0aa-44a7-9a38-7c9b17fbae2c" (page "3"))
+    (path "/eddb86bd-9206-456a-9ce6-a47edcb4b42b" (page "4"))
   )
   (symbol_instances
