File: hw/picocart64_v2/psram.kicad_sch (KiCad schematic)
At the start: 19 parts

Commit message: hw: v2 Finalize schematic
Parts:
- gave numbers to parts that had none: 19
Connections:
- net CS0 is gone; now on net CS1: U1.1 (~{CS}), U9.15 (O0)
- net CS1: no longer U2.1 (~{CS}), U9.14 (O1)
- net CS2: now also U2.1 (~{CS}), U9.14 (O1); no longer U3.1 (~{CS}), U9.13 (O2)
- net CS3: now also U3.1 (~{CS}), U9.13 (O2); no longer U4.1 (~{CS}), U9.12 (O3)
- net CS4: now also U4.1 (~{CS}), U9.12 (O3); no longer U5.1 (~{CS}), U9.11 (O4)
- net CS5: now also U5.1 (~{CS}), U9.11 (O4); no longer U6.1 (~{CS}), U9.10 (O5)
- net CS6: now also U6.1 (~{CS}), U9.10 (O5); no longer U7.1 (~{CS}), U9.9 (O6)
- net CS7: now also U7.1 (~{CS}), U9.9 (O6); no longer U8.1 (~{CS}), U9.7 (O7)
- new net CS8: U8.1 (~{CS}), U9.7 (O7)

Commit message: hw: Routing progress
Parts:
- added JP4, JP5: SolderJumper_2_Bridged, picocart64:SolderJumper-2_Small_Closed, symbol Jumper:SolderJumper_2_Bridged
- C1, C2, C3, C4, C5, C6, C7, C8, C9: footprint (none) -> Capacitor_SMD:C_0402_1005Metric
- R1: footprint (none) -> Resistor_SMD:R_0402_1005Metric
Connections:
- net GND: now also JP4.1 (A), JP5.1 (A); no longer U9.4 (E1), U9.5 (E2)
- new net: JP5.2 (B), U9.4 (E1)
- new net: JP4.2 (B), U9.5 (E2)
Other:
- moved on the sheet: R1
