File: hw/picocart64_v2/picocart64_v2.kicad_pcb (KiCad board)
At the start: 4 copper layers, 100 x 60 mm, 18 parts, among them J1 USB_C_Receptacle_USB2.0, J2 Conn_01x05, J3 Conn_02x06_Odd_Even, J4 Micro_SD_Card_Det, Q1 BSS84, SW1 BootButton, U3 RP2040_Stamp, U4 N64-Cartridge

Commit message: hw: v2 Finalize schematic
Parts:
- removed J1: USB_C_Receptacle_USB2.0, Connector_USB_Extra:USB_C_Receptacle_GT-USB-7010
- removed J2: Conn_01x05, Connector_PinHeader_2.54mm:PinHeader_1x05_P2.54mm_Vertical
- removed J3: Conn_02x06_Odd_Even, Connector_PinSocket_2.54mm:PinSocket_2x06_P2.54mm_Horizontal
- removed JP1, JP2, JP3, JP4: SolderJumper_2_Open, Jumper:SolderJumper-2_P1.3mm_Open_TrianglePad1.0x1.5mm
- removed R1: 1M, Resistor_SMD:R_0603_1608Metric
- added D1: WS2812B-2020, LED_SMD_Extra:WS2812B-2020, F.Cu at (266.8, 155.4)
- added R5: 5k1, Resistor_SMD:R_0603_1608Metric, F.Cu at (281.8, 128.1)
- added R6: 5k1, Resistor_SMD:R_0603_1608Metric, F.Cu at (274.3, 137.9)
- added RN1: 22R_x4, Resistor_SMD:R_Array_Convex_4x0603, F.Cu at (268.2, 141.0)
- added RN2: 22R_x4, Resistor_SMD:R_Array_Convex_4x0603, F.Cu at (262.8, 146.5)
- added RN3: 22R_x4, Resistor_SMD:R_Array_Convex_4x0603, F.Cu at (274.4, 134.2)
- added RN4: 22R_x4, Resistor_SMD:R_Array_Convex_4x0603, F.Cu at (264.0, 141.0)
- added RN5: 22R_x4, Resistor_SMD:R_Array_Convex_4x0603, F.Cu at (258.6, 146.5)
- added RN6: 22R_x4, Resistor_SMD:R_Array_Convex_4x0603, F.Cu at (254.5, 146.5)
- added U1: LY68L6400SLIT, Package_SO:SOIC-8_5.275x5.275mm_P1.27mm, F.Cu at (227.4, 130.2)
- added U10: USBLC6-2SC6, Package_TO_SOT_SMD:SOT-23-6, F.Cu at (249.8, 146.4)
- added U13: W25Q128JVS, Package_SO:SOIC-8_5.23x5.23mm_P1.27mm, F.Cu at (267.1, 135.2)
- added U16: ESP32-C3-WROOM-02, Espressif:ESP32-C3-WROOM-02, F.Cu at (247.8, 76.0)
- added U2: LY68L6400SLIT, Package_SO:SOIC-8_5.275x5.275mm_P1.27mm, F.Cu at (228.6, 137.1)
- added U5: LY68L6400SLIT, Package_SO:SOIC-8_5.275x5.275mm_P1.27mm, F.Cu at (218.2, 137.1)
- added U6: LY68L6400SLIT, Package_SO:SOIC-8_5.275x5.275mm_P1.27mm, F.Cu at (207.9, 142.2)
- added U7: LY68L6400SLIT, Package_SO:SOIC-8_5.275x5.275mm_P1.27mm, F.Cu at (218.2, 143.9)
- added U8: LY68L6400SLIT, Package_SO:SOIC-8_5.275x5.275mm_P1.27mm, F.Cu at (228.6, 143.9)
- added U9: SN74LVC138AQDRQ1, Package_SO:SOP-16_4.4x10.4mm_P1.27mm, F.Cu at (207.3, 132.8)
- Q1: value BSS84 -> FDN340P
- R2, R3: value 5k1 -> 1M
- U3: value RP2040_Stamp -> LY68L6400SLIT; footprint RP2040_Stamp:RP2040_Stamp_FlexyPin -> Package_SO:SOIC-8_5.275x5.275mm_P1.27mm
- U4: value N64-Cartridge -> LY68L6400SLIT; footprint picocart64:N64-Connector -> Package_SO:SOIC-8_5.275x5.275mm_P1.27mm; moved to F.Cu
- moved R2 184.3 mm to (278.5, 132.5), turned to 0 degrees
- moved R3 182.0 mm to (278.5, 135.0)
- moved Q1 170.1 mm to (277.4, 129.0)
- moved FB1 169.6 mm to (266.8, 144.6)
- moved SW1 152.1 mm to (268.4, 129.3)
- moved J4 106.8 mm to (254.6, 137.1)
- moved U3 101.1 mm to (237.7, 130.2)
- moved U4 68.2 mm to (217.0, 130.2), turned to 0 degrees
Connections:
- FB1 pad 1: /VBUS_unf -> /Mainboard/VBUS'
- J4 pad 1: /PMOD_5_SIO2 -> /Mainboard/SD_DAT2
- J4 pad 10: /PMOD_7_CS0 -> /Mainboard/SD_DET
- J4 pad 2: /PMOD_6_SIO3 -> /Mainboard/SD_DAT3
- J4 pad 3: /PMOD_1_SS -> /Mainboard/SD_CMD
- J4 pad 5: /PMOD_4_SCLK -> /Mainboard/SD_CLK
- J4 pad 7: /PMOD_2_SIO0 -> /Mainboard/SD_DAT0
- J4 pad 8: /PMOD_3_SIO1 -> /Mainboard/SD_DAT1
- Q1 pad 1: VBUS -> /Mainboard/3V3_USB
- Q1 pad 3: /N64_VCC -> /Mainboard/N64_VCC
- R2 pad 1: Net-(J1-PadA5) -> GND
- R2 pad 2: GND -> Net-(J1-PadS1)
- R3 pad 1: Net-(J1-PadB5) -> GND
- R3 pad 2: GND -> Net-(J2-PadS1)
- SW1 pad 1: GND -> /Mainboard/~{SSI_CS}
- SW1 pad 2: Net-(SW1-Pad2) -> Net-(R17-Pad1)
- U3 pad 1: /AD0 -> /PSRAM Array/CS2
- U3 pad 2: /AD1 -> /Mainboard/SSI_SD1
- U3 pad 3: /AD2 -> /Mainboard/SSI_SD2
- U3 pad 4: /AD3 -> GND
- U3 pad 5: /AD4 -> /Mainboard/SSI_SD0
- U3 pad 6: /AD5 -> /Mainboard/SSI_SCLK
- U3 pad 7: /AD6 -> /Mainboard/SSI_SD3
- U3 pad 8: /AD7 -> +3V3
- U4 pad 1: GND -> /PSRAM Array/CS3
- U4 pad 2: GND -> /Mainboard/SSI_SD1
- U4 pad 3: /AD15 -> /Mainboard/SSI_SD2
- U4 pad 4: /AD14 -> GND
- U4 pad 5: /AD13 -> /Mainboard/SSI_SD0
- U4 pad 6: GND -> /Mainboard/SSI_SCLK
- U4 pad 7: /AD12 -> /Mainboard/SSI_SD3
- U4 pad 8: /~{WRITE} -> +3V3
Routing:
- net (no net): track 0.00 -> 2025.8 mm, vias 0 -> 70
- net /N64_S_DAT: track 106.8 -> 0.00 mm, vias 3 -> 0
- net /N64_VCC: track 96.4 -> 0.00 mm, vias 5 -> 0
- net /N64_INT: track 87.7 -> 0.00 mm, vias 4 -> 0
- net /N64_NMI: track 76.4 -> 0.00 mm, vias 4 -> 0
- net /N64_SI_CLK: track 72.6 -> 0.00 mm, vias 5 -> 0
- net /AD0: track 70.6 -> 0.00 mm, vias 1 -> 0
- net /PMOD_6_SIO3: track 66.8 -> 0.00 mm, vias 2 -> 0
- net /PMOD_5_SIO2: track 65.6 -> 0.00 mm, vias 2 -> 0
- net /AD2: track 63.4 -> 0.00 mm, vias 1 -> 0
- net /AD1: track 63.1 -> 0.00 mm, vias 1 -> 0
- net /AD4: track 58.6 -> 0.00 mm, vias 1 -> 0
- net /N64_COLD_RESET: track 58.5 -> 0.00 mm, vias 3 -> 0
- net /AD3: track 58.3 -> 0.00 mm, vias 1 -> 0
- net /PMOD_4_SCLK: track 57.5 -> 0.00 mm, vias 1 -> 0
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- added copper zone on F.Cu, net (none)
- added copper zone on In1.Cu, net (none)
- removed copper zone on F.Cu, net /VBUS_unf
- removed copper zone on In1.Cu, net /VBUS_unf

Commit message: hw: Routing progress
Parts:
- added C1: 100n, Capacitor_SMD:C_0402_1005Metric, F.Cu at (113.0, 85.2)
- added C10: 10u, Capacitor_SMD:C_0603_1608Metric, F.Cu at (120.6, 74.2)
- added C11: 10u, Capacitor_SMD:C_0603_1608Metric, F.Cu at (122.9, 79.5)
- added C12: 12p, Capacitor_SMD:C_0402_1005Metric, F.Cu at (219.4, 101.2)
- added C13: 12p, Capacitor_SMD:C_0402_1005Metric, F.Cu at (226.8, 96.6)
- added C14: 100n, Capacitor_SMD:C_0402_1005Metric, F.Cu at (226.8, 94.7)
- added C15: 100n, Capacitor_SMD:C_0402_1005Metric, F.Cu at (229.6, 94.6)
- added C16: 100n, Capacitor_SMD:C_0402_1005Metric, F.Cu at (233.6, 88.7)
- added C17: 100n, Capacitor_SMD:C_0402_1005Metric, F.Cu at (225.2, 100.6)
- added C18: 100n, Capacitor_SMD:C_0402_1005Metric, F.Cu at (236.4, 88.7)
- added C19: 100n, Capacitor_SMD:C_0402_1005Metric, F.Cu at (218.3, 104.0)
- added C2: 100n, Capacitor_SMD:C_0402_1005Metric, F.Cu at (113.0, 92.8)
- added C20: 1u, Capacitor_SMD:C_0402_1005Metric, F.Cu at (221.2, 104.6)
- added C21: 100n, Capacitor_SMD:C_0402_1005Metric, F.Cu at (230.7, 88.7)
- added C22: 100n, Capacitor_SMD:C_0402_1005Metric, F.Cu at (215.4, 104.0)
- added C23: 1u, Capacitor_SMD:C_0402_1005Metric, F.Cu at (225.2, 98.6)
- added C24: 1u, Capacitor_SMD:C_0402_1005Metric, F.Cu at (223.9, 96.6)
- added C25: 100n, Capacitor_SMD:C_0402_1005Metric, F.Cu at (222.3, 102.7)
- added C26: 12p, Capacitor_SMD:C_0402_1005Metric, F.Cu at (232.5, 94.6)
- added C27: 12p, Capacitor_SMD:C_0402_1005Metric, F.Cu at (229.6, 96.6)
- added C28: 100n, Capacitor_SMD:C_0402_1005Metric, F.Cu at (229.2, 92.7)
- added C29: 100n, Capacitor_SMD:C_0402_1005Metric, F.Cu at (222.3, 98.7)
- added C3: 100n, Capacitor_SMD:C_0402_1005Metric, F.Cu at (122.6, 85.2)
- added C30: 100n, Capacitor_SMD:C_0402_1005Metric, F.Cu at (229.2, 90.7)
- added C31: 100n, Capacitor_SMD:C_0402_1005Metric, F.Cu at (226.2, 92.7)
- added C32: 100n, Capacitor_SMD:C_0402_1005Metric, F.Cu at (223.9, 94.7)
- added C33: 100n, Capacitor_SMD:C_0402_1005Metric, F.Cu at (219.4, 99.3)
- added C34: 1u, Capacitor_SMD:C_0402_1005Metric, F.Cu at (234.9, 90.7)
- added C35: 100n, Capacitor_SMD:C_0402_1005Metric, F.Cu at (232.0, 92.7)
- added C36: 100n, Capacitor_SMD:C_0402_1005Metric, F.Cu at (232.0, 90.7)
- added C37: 1u, Capacitor_SMD:C_0402_1005Metric, F.Cu at (222.3, 100.7)
- added C38: 10u, Capacitor_SMD:C_0603_1608Metric, F.Cu at (122.9, 81.3)
- added C39: 100n, Capacitor_SMD:C_0402_1005Metric, F.Cu at (112.9, 100.3)
- added C4: 100n, Capacitor_SMD:C_0402_1005Metric, F.Cu at (122.6, 92.8)
- added C5: 100n, Capacitor_SMD:C_0402_1005Metric, F.Cu at (132.3, 85.2)
- added C6: 100n, Capacitor_SMD:C_0402_1005Metric, F.Cu at (132.3, 92.8)
- added C7: 100n, Capacitor_SMD:C_0402_1005Metric, F.Cu at (141.9, 85.2)
- added C8: 100n, Capacitor_SMD:C_0402_1005Metric, F.Cu at (141.9, 92.8)
- added C9: 100n, Capacitor_SMD:C_0402_1005Metric, F.Cu at (229.0, 104.6)
- added J1: USB_C_Receptacle_USB2.0, Connector_USB_Extra:USB_C_Receptacle_GT-USB-7010, F.Cu at (104.4, 67.9)
- added J2: USB_C_Receptacle_USB2.0, Connector_USB_Extra:USB_C_Receptacle_GT-USB-7010, F.Cu at (104.4, 78.0)
- added J3: Conn_02x06_Odd_Even, Connector_PinHeader_2.54mm:PinHeader_2x06_P2.54mm_Vertical_SMD, B.Cu at (169.3, 66.8)
- added JP1: SolderJumper_2_Open, picocart64:SolderJumper-2_Small_Open, F.Cu at (172.2, 91.6)
- added JP2: SolderJumper_2_Bridged, picocart64:SolderJumper-2_Small_Closed, F.Cu at (181.0, 71.9)
- added JP3: SolderJumper_2_Bridged, picocart64:SolderJumper-2_Small_Closed, F.Cu at (181.0, 70.3)
- added JP4: SolderJumper_2_Bridged, picocart64:SolderJumper-2_Small_Closed, F.Cu at (121.7, 109.4)
- added JP5: SolderJumper_2_Bridged, picocart64:SolderJumper-2_Small_Closed, F.Cu at (119.4, 109.4)
- added R1: 10K, Resistor_SMD:R_0402_1005Metric, F.Cu at (226.1, 104.6)
- added R10: 22R, Resistor_SMD:R_0402_1005Metric, F.Cu at (111.0, 81.0)
- added R11: 22R, Resistor_SMD:R_0402_1005Metric, F.Cu at (111.0, 82.0)
- added R12: 10K, Resistor_SMD:R_0402_1005Metric, F.Cu at (221.0, 94.8)
- added R13: 10k, Resistor_SMD:R_0402_1005Metric, F.Cu at (224.9, 88.7)
- added R14: 22R, Resistor_SMD:R_0402_1005Metric, F.Cu at (213.6, 102.0)
- added R15: 22R, Resistor_SMD:R_0402_1005Metric, F.Cu at (216.6, 102.0)
- added R16: 470R, Resistor_SMD:R_0402_1005Metric, F.Cu at (216.6, 100.0)
- added R17: 1K, Resistor_SMD:R_0402_1005Metric, F.Cu at (114.6, 62.7)
- added R18: 10k, Resistor_SMD:R_0402_1005Metric, F.Cu at (218.1, 97.3)
- added R19: 10k, Resistor_SMD:R_0402_1005Metric, F.Cu at (213.6, 100.0)
- added R20: 100k, Resistor_SMD:R_0402_1005Metric, F.Cu at (122.9, 73.9)
- added R4: 22R, Resistor_SMD:R_0402_1005Metric, F.Cu at (134.0, 106.7)
- added R7: 10K, Resistor_SMD:R_0402_1005Metric, F.Cu at (218.1, 95.3)
- added R8: 22R, Resistor_SMD:R_0402_1005Metric, F.Cu at (132.7, 106.7)
- added R9: 10K, Resistor_SMD:R_0402_1005Metric, F.Cu at (226.3, 90.7)
- added TP1: TP_MCU2_SCK, TestPoint:TestPoint_Pad_D1.0mm, F.Cu at (206.7, 104.1)
- added TP2: TP_MCU2_CS, TestPoint:TestPoint_Pad_D1.0mm, F.Cu at (215.1, 97.5)
- added TP3: TP_MCU2_DIO, TestPoint:TestPoint_Pad_D1.0mm, F.Cu at (210.7, 101.6)
- added U11: AZ1117-3.3, Package_TO_SOT_SMD:SOT-223, F.Cu at (114.5, 76.7)
- added U12: N64-Cartridge, picocart64:N64-Connector, B.Cu at (150.2, 116.3)
- added U14: RP2040, Package_DFN_QFN_Extra:QFN-56_EP_7x7_Pitch0.4mm, F.Cu at (157.3, 95.1)
- added U15: RP2040, Package_DFN_QFN_Extra:QFN-56_EP_7x7_Pitch0.4mm, F.Cu at (142.0, 75.3)
- added Y1: 12MHz 10ppm, Crystal:Crystal_SMD_2520-4Pin_2.5x2.0mm, F.Cu at (169.7, 90.5)
- added Y2: 12MHz 10ppm, Crystal:Crystal_SMD_2520-4Pin_2.5x2.0mm, F.Cu at (152.4, 65.5)
- R2, R3: value 1M -> 100k; footprint Resistor_SMD:R_0603_1608Metric -> Resistor_SMD:R_0402_1005Metric
- R5, R6: footprint Resistor_SMD:R_0603_1608Metric -> Resistor_SMD:R_0402_1005Metric
- RN1, RN2, RN3, RN4, RN5, RN6: footprint Resistor_SMD:R_Array_Convex_4x0603 -> Resistor_SMD:R_Array_Convex_4x0402
- moved R5 188.9 mm to (105.1, 61.3), turned to 90 degrees
- moved R6 186.8 mm to (103.9, 61.3), turned to 90 degrees
- moved R2 186.2 mm to (106.4, 61.3), turned to -90 degrees
- moved D1 181.4 mm to (111.5, 61.7)
- moved R3 178.6 mm to (107.3, 83.9), turned to 180 degrees
- moved FB1 170.0 mm to (114.2, 69.9)
- moved Q1 162.5 mm to (123.4, 76.9)
- moved SW1 161.7 mm to (121.3, 62.3), turned to 180 degrees
- moved U13 160.8 mm to (109.4, 104.0)
- moved U10 156.1 mm to (115.2, 67.4)
- moved U2 125.9 mm to (109.4, 96.4)
- moved U3 125.5 mm to (119.2, 88.8)
- moved U1 125.0 mm to (109.4, 88.8)
- moved RN3 121.7 mm to (155.8, 106.7), turned to -90 degrees
- moved RN6 112.0 mm to (149.7, 106.7), turned to -90 degrees
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Connections:
- RN4 pad 1: /Mainboard/AD0' -> /Mainboard/AD0
- RN4 pad 2: /Mainboard/AD1' -> /Mainboard/AD1
- RN4 pad 3: /Mainboard/AD2' -> /Mainboard/AD2
- RN4 pad 4: /Mainboard/AD3' -> /Mainboard/AD3
- RN4 pad 5: /Mainboard/AD3 -> /Mainboard/AD3'
- RN4 pad 6: /Mainboard/AD2 -> /Mainboard/AD2'
- RN4 pad 7: /Mainboard/AD1 -> /Mainboard/AD1'
- RN4 pad 8: /Mainboard/AD0 -> /Mainboard/AD0'
- RN5 pad 1: /Mainboard/ALEL' -> /Mainboard/ALEL
- RN5 pad 2: /Mainboard/ALEH' -> /Mainboard/ALEH
- RN5 pad 3: /Mainboard/AD4' -> /Mainboard/AD4
- RN5 pad 4: /Mainboard/AD5' -> /Mainboard/AD5
- RN5 pad 5: /Mainboard/AD5 -> /Mainboard/AD5'
- RN5 pad 6: /Mainboard/AD4 -> /Mainboard/AD4'
- RN5 pad 7: /Mainboard/ALEH -> /Mainboard/ALEH'
- RN5 pad 8: /Mainboard/ALEL -> /Mainboard/ALEL'
- RN6 pad 1: /Mainboard/AD6' -> /Mainboard/AD7
- RN6 pad 2: /Mainboard/AD7' -> /Mainboard/AD6
- RN6 pad 3: /Mainboard/CIC_DCLK' -> /Mainboard/CIC_DCLK
- RN6 pad 4: /Mainboard/~{INT1'} -> /Mainboard/~{INT1}
- RN6 pad 5: /Mainboard/~{INT1} -> /Mainboard/~{INT1'}
- RN6 pad 6: /Mainboard/CIC_DCLK -> /Mainboard/CIC_DCLK'
- RN6 pad 7: /Mainboard/AD7 -> /Mainboard/AD6'
- RN6 pad 8: /Mainboard/AD6 -> /Mainboard/AD7'
- U1 pad 1: /PSRAM Array/CS0 -> /PSRAM Array/CS1
- U16 pad 11: /Mainboard/ESP32_D0_TX -> Net-(JP2-Pad1)
- U16 pad 12: /Mainboard/ESP32_D1_RX -> Net-(JP3-Pad1)
- U2 pad 1: /PSRAM Array/CS1 -> /PSRAM Array/CS2
- U3 pad 1: /PSRAM Array/CS2 -> /PSRAM Array/CS3
- U4 pad 1: /PSRAM Array/CS3 -> /PSRAM Array/CS4
- U5 pad 1: /PSRAM Array/CS4 -> /PSRAM Array/CS5
- U6 pad 1: /PSRAM Array/CS5 -> /PSRAM Array/CS6
- U7 pad 1: /PSRAM Array/CS6 -> /PSRAM Array/CS7
- U8 pad 1: /PSRAM Array/CS7 -> /PSRAM Array/CS8
- U9 pad 10: /PSRAM Array/CS5 -> /PSRAM Array/CS6
- U9 pad 11: /PSRAM Array/CS4 -> /PSRAM Array/CS5
- U9 pad 12: /PSRAM Array/CS3 -> /PSRAM Array/CS4
- U9 pad 13: /PSRAM Array/CS2 -> /PSRAM Array/CS3
- U9 pad 14: /PSRAM Array/CS1 -> /PSRAM Array/CS2
- U9 pad 15: /PSRAM Array/CS0 -> /PSRAM Array/CS1
- U9 pad 4: GND -> Net-(JP5-Pad2)
- U9 pad 5: GND -> Net-(JP4-Pad2)
- U9 pad 7: /PSRAM Array/CS7 -> /PSRAM Array/CS8
- U9 pad 9: /PSRAM Array/CS6 -> /PSRAM Array/CS7
Routing:
- net (no net): track 2025.8 -> 0.00 mm, vias 70 -> 0
- net /Mainboard/SSI_SD2: track 0.00 -> 104.4 mm, vias 0 -> 5
- net /Mainboard/SSI_SD1: track 0.00 -> 102.6 mm, vias 0 -> 2
- net /Mainboard/SSI_SCLK: track 0.00 -> 97.5 mm, vias 0 -> 5
- net /Mainboard/SSI_SD3: track 0.00 -> 95.9 mm, vias 0 -> 5
- net /Mainboard/SSI_SD0: track 0.00 -> 94.1 mm, vias 0 -> 5
- net /Mainboard/N64_VCC: track 0.00 -> 91.0 mm, vias 0 -> 5
- net +3V3: track 131.0 -> 183.1 mm, vias 2 -> 14
- net /Mainboard/~{SSI_CS}: track 0.00 -> 50.4 mm
- net Net-(R10-Pad2): track 0.00 -> 49.1 mm
- net Net-(R11-Pad2): track 0.00 -> 48.9 mm
- net GND: track 86.3 -> 124.8 mm, vias 71 -> 51
- net VBUS: track 49.2 -> 13.6 mm
- net /Mainboard/CIC_DIO: track 0.00 -> 33.5 mm, vias 0 -> 1
- net /Mainboard/DEMUX_A0: track 0.00 -> 31.4 mm
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- added copper zone on F.Cu, net /Mainboard/3V3_USB
- added copper zone on F.Cu, net /Mainboard/VBUS'
- added copper zone on In1.Cu, net /Mainboard/VBUS'
- removed copper zone on F.Cu, net (none)
- removed copper zone on In1.Cu, net (none)
Other:
- board text added: "4 Layers 1.00 mm thickness 6/6 mil traces 45 deg. chamfered gold-plated edge connector"
- board text removed: "+"
- board text removed: "+3V3"
- board text removed: "1. ~{SS}"
- board text removed: "2. SIO0"
- board text removed: "3. SIO1"
- board text removed: "4. SCLK"
- board text removed: "5. SIO2"
- board text removed: "6. SIO3"
- board text removed: "7. ~{CS0}"
- board text removed: "8. N/C"
- board text removed: "C"
- board text removed: "D"
- board text removed: "G"
- board text removed: "GND"
- board text removed: "INT"
- board text removed: "NMI"
- board text removed: "R"
- board text removed: "SI_CLK"
- board text removed: "SWCLK"
- board text removed: "SWDIO"
- board text removed: "S_DAT"
- board text removed: "~{RST}"

Commit message: hw: More routing progress
Parts:
- moved Y1 4.44 mm to (167.9, 94.6), turned to 0 degrees
- moved JP1 3.45 mm to (168.8, 91.9), turned to -90 degrees
Routing:
- net /Mainboard/SI_DAT: track 0.00 -> 42.9 mm, vias 0 -> 2
- net /Mainboard/~{READ}: track 0.00 -> 20.8 mm, vias 0 -> 2
- net /Mainboard/~{WRITE}: track 0.00 -> 17.9 mm, vias 0 -> 2
- net /Mainboard/MCU1_XIN: track 0.00 -> 11.3 mm
- net Net-(C21-Pad1): track 0.00 -> 7.88 mm, vias 0 -> 1
- net /Mainboard/MCU1_XOUT: track 0.00 -> 6.32 mm
- net /Mainboard/~{COLD_RESET}: track 27.9 -> 31.4 mm
- net GND: track 124.8 -> 128.1 mm, vias 51 -> 58
- net /Mainboard/CIC_DCLK: track 30.1 -> 28.7 mm
- net /Mainboard/AD4: track 15.9 -> 14.9 mm
- net /Mainboard/CIC_DIO: track 33.5 -> 34.3 mm
- net /Mainboard/AD2: track 23.7 -> 23.0 mm
- net /Mainboard/SSI_SD2: track 104.4 -> 103.7 mm
- net /Mainboard/AD7: track 13.9 -> 14.5 mm
- net /Mainboard/AD0: track 24.2 -> 23.6 mm
